File: diagram_chart.kicad_sch (KiCad schematic)
At the start: 10 parts, among them U2 74HC165

Commit message: Added the things I said I would
Parts:
- added HDSP-7513_red, HDSP-7803_green: HDSP-7503, Display_7Segment:HDSP-A151, symbol Display_Character:HDSP-7503
- added J1: Barrel_Jack, Connector_BarrelJack:BarrelJack_CUI_PJ-102AH_Horizontal, symbol Connector:Barrel_Jack
- added SW1: SW_SPDT, switch:SW_Toggle_Blue_wSlots, symbol Switch:SW_SPDT
Changed lines of the file:
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@@
 (kicad_sch (version 20230121) (generator eeschema)
   (paper "A4")
+  (symbol (lib_id "Switch:SW_SPDT") (at 252.73 143.51 0) (unit 1)
+    (in_bom yes) (on_board yes) (dnp no) (fields_autoplaced)
+    (property "Reference" "SW1" (at 252.73 134.62 0)
+      (effects (font (size 1.27 1.27)))
+    )
+    (property "Value" "SW_SPDT" (at 252.73 137.16 0)
+      (effects (font (size 1.27 1.27)))
+    )
+    (property "Footprint" "switch:SW_Toggle_Blue_wSlots" (at 252.73 143.51 0)
+      (effects (font (size 1.27 1.27)) hide)
+    )
+    (property "Datasheet" "~" (at 252.73 151.13 0)
+      (effects (font (size 1.27 1.27)) hide)
+    )
+    (pin "1")
+    (pin "3")
+    (pin "2")
+    (instances
+      (project "diagram_chart"
+        (path "/6dfb841c-0ebb-4587-a5cf-7b85233b045b"
+          (reference "SW1") (unit 1)
+        )
+      )
+    )
+  )
+  (symbol (lib_id "Connector:Barrel_Jack") (at 81.28 55.88 0) (unit 1)
+    (in_bom yes) (on_board yes) (dnp no) (fields_autoplaced)
+    (property "Reference" "J1" (at 81.28 46.99 0)
+      (effects (font (size 1.27 1.27)))
+    )
+    (property "Value" "Barrel_Jack" (at 81.28 49.53 0)
+      (effects (font (size 1.27 1.27)))
+    )
+    (property "Footprint" "Connector_BarrelJack:BarrelJack_CUI_PJ-102AH_Horizontal" (at 82.55 56.896 0)
+      (effects (font (size 1.27 1.27)) hide)
+    )
+    (property "Datasheet" "~" (at 82.55 56.896 0)
+      (effects (font (size 1.27 1.27)) hide)
+    )
+    (pin "1")
+    (pin "2")
+    (instances
+      (project "diagram_chart"
+        (path "/6dfb841c-0ebb-4587-a5cf-7b85233b045b"
+          (reference "J1") (unit 1)
+        )
+      )
+    )
+  )
   (symbol (lib_id "74xx:74HC165") (at 71.12 114.3 0) (unit 1)
     (in_bom yes) (on_board yes) (dnp no) (fields_autoplaced)
@@
         )
       )
+    )
+  )
+  (symbol (lib_id "Display_Character:HDSP-7503") (at 88.9 171.45 0) (unit 1)
+    (in_bom yes) (on_board yes) (dnp no) (fields_autoplaced)
+    (property "Reference" "HDSP-7513_red" (at 88.9 153.67 0)
+      (effects (font (size 1.27 1.27)))
+    )
+    (property "Value" "HDSP-7503" (at 88.9 156.21 0)
+      (effects (font (size 1.27 1.27)))
+    )
+    (property "Footprint" "Display_7Segment:HDSP-A151" (at 88.9 185.42 0)
+      (effects (font (size 1.27 1.27)) hide)
+    )
+    (property "Datasheet" "https://docs.broadcom.com/docs/AV02-2553EN" (at 78.74 157.48 0)
+      (effects (font (size 1.27 1.27)) hide)
+    )
+    (pin "1")
+    (pin "4")
+    (pin "9")
+    (pin "2")
+    (pin "7")
+    (pin "8")
+    (pin "5")
+    (pin "10")
+    (pin "3")
+    (pin "6")
+    (instances
+      (project "diagram_chart"
+        (path "/6dfb841c-0ebb-4587-a5cf-7b85233b045b"
+          (reference "HDSP-7513_red") (unit 1)
+        )
+      )
+    )
+  )
+  (symbol (lib_id "Display_Character:HDSP-7503") (at 134.62 173.99 0) (unit 1)
+    (in_bom yes) (on_board yes) (dnp no) (fields_autoplaced)
+    (property "Reference" "HDSP-7803_green" (at 134.62 156.21 0)
+      (effects (font (size 1.27 1.27)))
+    )
+    (property "Value" "HDSP-7503" (at 134.62 158.75 0)
+      (effects (font (size 1.27 1.27)))
+    )
+    (property "Footprint" "Display_7Segment:HDSP-A151" (at 134.62 187.96 0)
+      (effects (font (size 1.27 1.27)) hide)
+    )
+    (property "Datasheet" "https://docs.broadcom.com/docs/AV02-2553EN" (at 124.46 160.02 0)
+      (effects (font (size 1.27 1.27)) hide)
+    )
+    (pin "1")
+    (pin "4")
+    (pin "9")
+    (pin "2")
+    (pin "7")
+    (pin "8")
+    (pin "5")
+    (pin "10")
+    (pin "3")
+    (pin "6")
+    (instances
+      (project "diagram_chart"
+        (path "/6dfb841c-0ebb-4587-a5cf-7b85233b045b"
+          (reference "HDSP-7803_green") (unit 1)
+        )
+      )

Commit message: Added screw terminals
Parts:
- added J2: Screw_Terminal_01x02, TerminalBlock_Phoenix:TerminalBlock_Phoenix_MPT-0,5-2-2.54_1x02_P2.54mm_Horizontal, symbol Connector:Screw_Terminal_01x02
Changed lines of the file:
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@@
+    )
+  )
+  (symbol (lib_id "Connector:Screw_Terminal_01x02") (at 46.99 82.55 0) (unit 1)
+    (in_bom yes) (on_board yes) (dnp no) (fields_autoplaced)
+    (property "Reference" "J2" (at 49.53 82.55 0)
+      (effects (font (size 1.27 1.27)) (justify left))
+    )
+    (property "Value" "Screw_Terminal_01x02" (at 49.53 85.09 0)
+      (effects (font (size 1.27 1.27)) (justify left))
+    )
+    (property "Footprint" "TerminalBlock_Phoenix:TerminalBlock_Phoenix_MPT-0,5-2-2.54_1x02_P2.54mm_Horizontal" (at 46.99 82.55 0)
+      (effects (font (size 1.27 1.27)) hide)
+    )
+    (property "Datasheet" "~" (at 46.99 82.55 0)
+      (effects (font (size 1.27 1.27)) hide)
+    )
+    (pin "1")
+    (pin "2")
+    (instances
+      (project "diagram_chart"
+        (path "/6dfb841c-0ebb-4587-a5cf-7b85233b045b"
+          (reference "J2") (unit 1)
+        )
+      )
     )
   )
