File: KiCad/diagram_chart.kicad_sch (KiCad schematic)
At the start: 79 parts, among them SW0 SW0, SW1 SW1, SW2 SW2, SW3 SW3, SW4 SW4, SW5 SW5, SW6 SW6, SW7 SW7, U1 TPIC6C595, U2 74HC165, Y1 16MHz

Commit message: Made 14x14 cm. Positioned and alligned switches, displays and LEDs. 1oZ coppar makes me decide for 1mm width per AMP Meaning 0,2mm is enough for 200mA
Parts:
- D0, D1, D2, D3, D4, D5, D6, D7: footprint LED_THT:LED_D5.0mm -> LED_THT:LED_D3.0mm
Changed lines of the file:
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@@
       (effects (font (size 1.27 1.27)))
     )
-    (property "Footprint" "LED_THT:LED_D5.0mm" (at 67.31 219.71 0)
+    (property "Footprint" "LED_THT:LED_D3.0mm" (at 67.31 219.71 0)
       (effects (font (size 1.27 1.27)) hide)
     )
@@
       (effects (font (size 1.27 1.27)))
     )
-    (property "Footprint" "LED_THT:LED_D5.0mm" (at 44.45 219.71 0)
+    (property "Footprint" "LED_THT:LED_D3.0mm" (at 44.45 219.71 0)
       (effects (font (size 1.27 1.27)) hide)
     )
@@
       (effects (font (size 1.27 1.27)))
     )
-    (property "Footprint" "LED_THT:LED_D5.0mm" (at 57.15 219.71 0)
+    (property "Footprint" "LED_THT:LED_D3.0mm" (at 57.15 219.71 0)
       (effects (font (size 1.27 1.27)) hide)
     )
@@
       (effects (font (size 1.27 1.27)))
     )
-    (property "Footprint" "LED_THT:LED_D5.0mm" (at 33.02 219.71 0)
+    (property "Footprint" "LED_THT:LED_D3.0mm" (at 33.02 219.71 0)
       (effects (font (size 1.27 1.27)) hide)
     )
@@
       (effects (font (size 1.27 1.27)))
     )
-    (property "Footprint" "LED_THT:LED_D5.0mm" (at 78.74 219.71 0)
+    (property "Footprint" "LED_THT:LED_D3.0mm" (at 78.74 219.71 0)
       (effects (font (size 1.27 1.27)) hide)
     )
@@
       (effects (font (size 1.27 1.27)))
     )
-    (property "Footprint" "LED_THT:LED_D5.0mm" (at 21.59 219.71 0)
+    (property "Footprint" "LED_THT:LED_D3.0mm" (at 21.59 219.71 0)
       (effects (font (size 1.27 1.27)) hide)
     )
@@
       (effects (font (size 1.27 1.27)))
     )
-    (property "Footprint" "LED_THT:LED_D5.0mm" (at 101.6 219.71 0)
+    (property "Footprint" "LED_THT:LED_D3.0mm" (at 101.6 219.71 0)
       (effects (font (size 1.27 1.27)) hide)
     )
@@
       (effects (font (size 1.27 1.27)))
     )
-    (property "Footprint" "LED_THT:LED_D5.0mm" (at 90.17 219.71 0)
-      (effects (font (size 1.27 1.27)) hide)
-    )
+    (property "Footprint" "LED_THT:LED_D3.0mm" (at 90.17 219.71 0)
+      (effects (font (size 1.27 1.27)) hide)
+    )
