File: KiCad/diagram_chart.kicad_sch (KiCad schematic)
At the start: 79 parts, among them SW0 SW0, SW1 SW1, SW2 SW2, SW3 SW3, SW4 SW4, SW5 SW5, SW6 SW6, SW7 SW7, U1 TPIC6C595, U2 74HC165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

Commit message: Fixed SPDT to correct sizes. Also flipped them so down is off. Added values of resistors, etc to silkscreen. Made the board 13x13 instead of 14x14. Centralized SPDT sw3, will after lunch center the rest accordingly.
Parts:
- SW0, SW1, SW2, SW3, SW4, SW5, SW6, SW7, SW_Mem1, SW_Serr1, SW__WR1: footprint switch:SW_Toggle_Blue_wSlots -> switch:SW_Toggle_Blue_SMALL
Connections:
- net at CU1.1, CU_Caps1.1, C_MCU1.1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: now also SW_Mem1.3 (C), SW__WR1.3 (C)
Changed lines of the file:
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@@
   (junction (at 165.1 110.49) (diameter 0) (color 0 0 0 0)
   )
+  (junction (at 332.74 63.5) (diameter 0) (color 0 0 0 0)
+  )
   (junction (at 72.39 163.83) (diameter 0) (color 0 0 0 0)
   )
@@
   (junction (at 405.13 186.69) (diameter 0.2) (color 0 0 0 1)
   )
+  (junction (at 332.74 40.64) (diameter 0) (color 0 0 0 0)
+  )
   (junction (at 349.25 58.42) (diameter 0) (color 0 0 0 0)
   )
@@
     (stroke (width 0.2) (type default) (color 255 0 0 1))
   )
+  (wire (pts (xy 321.31 40.64) (xy 332.74 40.64))
+    (stroke (width 0.2) (type default) (color 255 0 0 1))
+  )
   (wire (pts (xy 374.65 48.26) (xy 405.13 48.26))
     (stroke (width 0.2) (type default) (color 0 0 0 1))
@@
     (stroke (width 0.2) (type default) (color 0 0 0 1))
   )
+  (wire (pts (xy 332.74 63.5) (xy 332.74 83.82))
+    (stroke (width 0.2) (type default) (color 255 0 0 1))
+  )
   (wire (pts (xy 86.36 80.01) (xy 78.74 80.01))
     (stroke (width 0) (type default))
@@
     (stroke (width 0) (type default))
   )
+  (wire (pts (xy 321.31 63.5) (xy 332.74 63.5))
+    (stroke (width 0.2) (type default) (color 255 0 0 1))
+  )
   (wire (pts (xy 163.83 191.77) (xy 163.83 210.82))
     (stroke (width 0) (type default))
@@
     (stroke (width 0) (type default))
   )
-  (wire (pts (xy 332.74 16.51) (xy 332.74 83.82))
+  (wire (pts (xy 332.74 16.51) (xy 332.74 40.64))
     (stroke (width 0.2) (type default) (color 255 0 0 1))
   )
@@
     (stroke (width 0.2) (type default) (color 255 0 0 1))
   )
+  (wire (pts (xy 332.74 40.64) (xy 332.74 63.5))
+    (stroke (width 0.2) (type default) (color 255 0 0 1))
+  )
   (wire (pts (xy 91.44 35.56) (xy 80.01 35.56))
     (stroke (width 0) (type default))
@@
       (effects (font (size 1.27 1.27)))
     )
-    (property "Footprint" "switch:SW_Toggle_Blue_wSlots" (at 386.08 223.52 0)
+    (property "Footprint" "switch:SW_Toggle_Blue_SMALL" (at 386.08 223.52 0)
       (effects (font (size 1.27 1.27)) hide)
     )
@@
       (effects (font (size 1.27 1.27)))
     )
-    (property "Footprint" "switch:SW_Toggle_Blue_wSlots" (at 384.81 176.53 0)
+    (property "Footprint" "switch:SW_Toggle_Blue_SMALL" (at 384.81 176.53 0)
       (effects (font (size 1.27 1.27)) hide)
     )
@@
       (effects (font (size 1.27 1.27)))
     )
-    (property "Footprint" "switch:SW_Toggle_Blue_wSlots" (at 318.77 81.28 0)
+    (property "Footprint" "switch:SW_Toggle_Blue_SMALL" (at 318.77 81.28 0)
       (effects (font (size 1.27 1.27)) hide)
     )
@@
       (effects (font (size 1.27 1.27)))
     )
-    (property "Footprint" "switch:SW_Toggle_Blue_wSlots" (at 316.23 60.96 0)
+    (property "Footprint" "switch:SW_Toggle_Blue_SMALL" (at 316.23 60.96 0)
       (effects (font (size 1.27 1.27)) hide)
     )
@@
       (effects (font (size 1.27 1.27)))
     )
-    (property "Footprint" "switch:SW_Toggle_Blue_wSlots" (at 386.08 60.96 0)
+    (property "Footprint" "switch:SW_Toggle_Blue_SMALL" (at 386.08 60.96 0)
       (effects (font (size 1.27 1.27)) hide)
     )
@@
       (effects (font (size 1.27 1.27)))
     )
-    (property "Footprint" "switch:SW_Toggle_Blue_wSlots" (at 383.54 130.81 0)
+    (property "Footprint" "switch:SW_Toggle_Blue_SMALL" (at 383.54 130.81 0)
       (effects (font (size 1.27 1.27)) hide)
     )
@@
       (effects (font (size 1.27 1.27)))
     )
-    (property "Footprint" "switch:SW_Toggle_Blue_wSlots" (at 384.81 107.95 0)
+    (property "Footprint" "switch:SW_Toggle_Blue_SMALL" (at 384.81 107.95 0)
       (effects (font (size 1.27 1.27)) hide)
     )
@@
       (effects (font (size 1.27 1.27)))
     )
-    (property "Footprint" "switch:SW_Toggle_Blue_wSlots" (at 383.54 153.67 0)
+    (property "Footprint" "switch:SW_Toggle_Blue_SMALL" (at 383.54 153.67 0)
       (effects (font (size 1.27 1.27)) hide)
     )
@@
       (effects (font (size 1.27 1.27)))
     )
-    (property "Footprint" "switch:SW_Toggle_Blue_wSlots" (at 384.81 198.12 0)
+    (property "Footprint" "switch:SW_Toggle_Blue_SMALL" (at 384.81 198.12 0)
       (effects (font (size 1.27 1.27)) hide)
     )
@@
       (effects (font (size 1.27 1.27)))
     )
-    (property "Footprint" "switch:SW_Toggle_Blue_wSlots" (at 316.23 38.1 0)
+    (property "Footprint" "switch:SW_Toggle_Blue_SMALL" (at 316.23 38.1 0)
       (effects (font (size 1.27 1.27)) hide)
     )
@@
       (effects (font (size 1.27 1.27)))
     )
-    (property "Footprint" "switch:SW_Toggle_Blue_wSlots" (at 384.81 86.36 0)
+    (property "Footprint" "switch:SW_Toggle_Blue_SMALL" (at 384.81 86.36 0)
       (effects (font (size 1.27 1.27)) hide)
     )

Commit message: Will need to recheck ignored violations tomorrow. DRC checker seems fine. Hole PTH to copper is fine at 0.35mm, not at 0,55. But YOLO
Parts:
- added CU2: 100nF, Capacitor_THT:C_Disc_D3.0mm_W1.6mm_P2.50mm, symbol Device:C
- added R32: 330Ω, Resistor_THT:R_Axial_DIN0207_L6.3mm_D2.5mm_P7.62mm_Horizontal, symbol Device:R
- F1: value 1A -> 2A
- R0, R1, R2, R3, R4, R5, R6, R7: value 220Ω -> 330Ω
- SW_Mem1: value SW__Mem1 -> SW__MEM
- SW__WR1: value SW__WR1 -> SW__WR
Connections:
- net GND: now also CU2.2
- net at MCU_0.16 (PB2): now also R32.2; no longer RGB1.1 (Pin_1)
- net at MCU_0.21 (AREF): now also CU2.1
- new net: R32.1, RGB1.1 (Pin_1)
Changed lines of the file:
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@@
   (junction (at 238.76 87.63) (diameter 0) (color 0 0 0 0)
   )
+  (junction (at 297.18 99.06) (diameter 0) (color 0 0 0 0)
+  )
   (junction (at 57.15 231.14) (diameter 0) (color 0 0 0 0)
   )
@@
     (stroke (width 0) (type default))
   )
+  (wire (pts (xy 297.18 99.06) (xy 281.94 99.06))
+    (stroke (width 0.2) (type default) (color 0 0 0 1))
+  )
   (wire (pts (xy 80.01 35.56) (xy 80.01 73.66))
     (stroke (width 0) (type default))
@@
     (stroke (width 0) (type default))
   )
-  (wire (pts (xy 248.92 63.5) (xy 248.92 72.39))
+  (wire (pts (xy 248.92 63.5) (xy 248.92 64.77))
     (stroke (width 0) (type default))
   )
@@
     (stroke (width 0.2) (type default) (color 255 0 0 1))
   )
+  (wire (pts (xy 281.94 99.06) (xy 281.94 74.93))
+    (stroke (width 0.2) (type default) (color 0 0 0 1))
+  )
   (wire (pts (xy 243.84 110.49) (xy 243.84 113.03))
     (stroke (width 0) (type default))
@@
       (effects (font (size 1.27 1.27)))
     )
-    (property "Value" "220Ω" (at 95.25 31.75 90)
+    (property "Value" "330Ω" (at 95.25 31.75 90)
       (effects (font (size 1.27 1.27)))
     )
@@
       (effects (font (size 1.27 1.27)))
     )
-    (property "Value" "220Ω" (at 110.49 36.83 90)
+    (property "Value" "330Ω" (at 110.49 36.83 90)
       (effects (font (size 1.27 1.27)))
     )
@@
       (effects (font (size 1.27 1.27)))
     )
-    (property "Value" "220Ω" (at 95.25 41.91 90)
+    (property "Value" "330Ω" (at 95.25 41.91 90)
       (effects (font (size 1.27 1.27)))
     )
@@
       (effects (font (size 1.27 1.27)))
     )
-    (property "Value" "220Ω" (at 102.87 29.21 90)
+    (property "Value" "330Ω" (at 102.87 29.21 90)
       (effects (font (size 1.27 1.27)))
     )
@@
       (effects (font (size 1.27 1.27)))
     )
-    (property "Value" "220Ω" (at 115.57 44.45 90)
+    (property "Value" "330Ω" (at 115.57 44.45 90)
       (effects (font (size 1.27 1.27)))
     )
@@
       (effects (font (size 1.27 1.27)) (justify left))
     )
-    (property "Value" "1A" (at 217.17 46.99 0)
+    (property "Value" "2A" (at 217.17 46.99 0)
       (effects (font (size 1.27 1.27)) (justify left))
     )
@@
       (effects (font (size 1.27 1.27)))
     )
-    (property "Value" "SW__WR1" (at 316.23 54.61 0)
+    (property "Value" "SW__WR" (at 316.23 54.61 0)
       (effects (font (size 1.27 1.27)))
     )
@@
       (effects (font (size 1.27 1.27)))
     )
-    (property "Value" "220Ω" (at 116.84 34.29 90)
+    (property "Value" "330Ω" (at 116.84 34.29 90)
       (effects (font (size 1.27 1.27)))
     )
@@
       (effects (font (size 1.27 1.27)))
     )
-    (property "Value" "220Ω" (at 110.49 26.67 90)
+    (property "Value" "330Ω" (at 110.49 26.67 90)
       (effects (font (size 1.27 1.27)))
     )
@@
       (effects (font (size 1.27 1.27)))
     )
-    (property "Value" "220Ω" (at 102.87 39.37 90)
+    (property "Value" "330Ω" (at 102.87 39.37 90)
       (effects (font (size 1.27 1.27)))
     )
@@
     )
   )
+  (symbol (lib_id "Device:C") (at 281.94 71.12 0) (unit 1)
+    (in_bom yes) (on_board yes) (dnp no)
+    (property "Reference" "CU2" (at 285.75 69.85 0)
+      (effects (font (size 1.27 1.27)) (justify left))
+    )
+    (property "Value" "100nF" (at 285.75 72.39 0)
+      (effects (font (size 1.27 1.27)) (justify left))
+    )
+    (property "Footprint" "Capacitor_THT:C_Disc_D3.0mm_W1.6mm_P2.50mm" (at 282.9052 74.93 0)
+      (effects (font (size 1.27 1.27)) hide)
+    )
+    (property "Datasheet" "~" (at 281.94 71.12 0)
+      (effects (font (size 1.27 1.27)) hide)
+    )
+    (pin "2")
+    (pin "1")
+    (instances
+      (project "diagram_chart"
+        (path "/6dfb841c-0ebb-4587-a5cf-7b85233b045b"
+          (reference "CU2") (unit 1)
+        )
+      )
+    )
+  )
   (symbol (lib_id "TPIC6C595:TPIC6595") (at 134.62 40.64 0) (mirror y) (unit 1)
     (in_bom yes) (on_board yes) (dnp no)
@@
     )
   )
+  (symbol (lib_id "Device:R") (at 248.92 68.58 0) (unit 1)
+    (in_bom yes) (on_board yes) (dnp no)
+    (property "Reference" "R32" (at 246.38 68.58 0)
+      (effects (font (size 1.27 1.27)) (justify left))
+    )
+    (property "Value" "330Ω" (at 241.3 68.58 0)
+      (effects (font (size 1.27 1.27)) (justify left))
+    )
+    (property "Footprint" "Resistor_THT:R_Axial_DIN0207_L6.3mm_D2.5mm_P7.62mm_Horizontal" (at 247.142 68.58 90)
+      (effects (font (size 1.27 1.27)) hide)
+    )
+    (property "Datasheet" "~" (at 248.92 68.58 0)
+      (effects (font (size 1.27 1.27)) hide)
+    )
+    (pin "2")
+    (pin "1")
+    (instances
+      (project "diagram_chart"
+        (path "/6dfb841c-0ebb-4587-a5cf-7b85233b045b"
+          (reference "R32") (unit 1)
+        )
+      )
+    )
+  )
   (symbol (lib_id "Device:R") (at 373.38 182.88 0) (unit 1)
     (in_bom yes) (on_board yes) (dnp no) (fields_autoplaced)
@@
       (effects (font (size 1.27 1.27)))
     )
-    (property "Value" "SW__Mem1" (at 316.23 31.75 0)
+    (property "Value" "SW__MEM" (at 316.23 31.75 0)
       (effects (font (size 1.27 1.27)))
     )

Commit message: Verified the footprint seems ok. Ran DRC checker several times.
I can't claim to be certain of of anything, that would be jinxing.
But will cross my fingers and order the PCB this afternoon.
Parts:
- added NC1, NC2, NC3, NC4, RGB2: Screw Terminal, TerminalBlock_Phoenix:TerminalBlock_Phoenix_MPT-0,5-2-2.54_1x02_P2.54mm_Horizontal, symbol Connector:Screw_Terminal_01x02
- added R33: 330Ω, Resistor_THT:R_Axial_DIN0207_L6.3mm_D2.5mm_P7.62mm_Horizontal, symbol Device:R
- F1: footprint Fuse:Fuseholder_Clip-5x20mm_Keystone_3512_Inline_P23.62x7.27mm_D1.02x1.57mm_Horizontal -> Fuse:Fuseholder_Clip-5x20mm_Eaton_1A5601-01_Inline_P20.80x6.76mm_D1.70mm_Horizontal
Connections:
- net at MCU_0.16 (PB2), R32.2: now also R33.2
- new net: R33.1, RGB2.1 (Pin_1)
Changed lines of the file:
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@@
   (junction (at 73.66 138.43) (diameter 0) (color 0 0 0 0)
   )
+  (junction (at 248.92 72.39) (diameter 0) (color 0 0 0 0)
+  )
   (junction (at 297.18 135.89) (diameter 0.2) (color 0 0 0 1)
   )
@@
     (stroke (width 0.2) (type default) (color 255 0 0 1))
   )
+  (wire (pts (xy 232.41 71.12) (xy 248.92 71.12))
+    (stroke (width 0) (type default))
+  )
   (wire (pts (xy 374.65 48.26) (xy 405.13 48.26))
     (stroke (width 0.2) (type default) (color 0 0 0 1))
@@
     (stroke (width 0) (type default))
   )
+  (wire (pts (xy 232.41 66.04) (xy 232.41 71.12))
+    (stroke (width 0) (type default))
+  )
   (wire (pts (xy 147.32 35.56) (xy 152.4 35.56))
     (stroke (width 0.3) (type default) (color 255 255 0 1))
@@
     (stroke (width 0.2) (type default) (color 255 0 0 1))
   )
+  (wire (pts (xy 248.92 71.12) (xy 248.92 72.39))
+    (stroke (width 0) (type default))
+  )
   (wire (pts (xy 246.38 40.64) (xy 246.38 16.51))
     (stroke (width 0.2) (type default) (color 255 0 0 1))
@@
     (stroke (width 0.2) (type default) (color 0 0 0 1))
   )
+  (wire (pts (xy 232.41 57.15) (xy 232.41 58.42))
+    (stroke (width 0) (type default))
+  )
   (wire (pts (xy 151.13 130.81) (xy 165.1 130.81))
     (stroke (width 0.2) (type default) (color 0 0 0 1))
@@
     )
   )
+  (symbol (lib_id "Device:R") (at 232.41 62.23 0) (unit 1)
+    (in_bom yes) (on_board yes) (dnp no)
+    (property "Reference" "R33" (at 229.87 62.23 0)
+      (effects (font (size 1.27 1.27)) (justify left))
+    )
+    (property "Value" "330Ω" (at 224.79 62.23 0)
+      (effects (font (size 1.27 1.27)) (justify left))
+    )
+    (property "Footprint" "Resistor_THT:R_Axial_DIN0207_L6.3mm_D2.5mm_P7.62mm_Horizontal" (at 230.632 62.23 90)
+      (effects (font (size 1.27 1.27)) hide)
+    )
+    (property "Datasheet" "~" (at 232.41 62.23 0)
+      (effects (font (size 1.27 1.27)) hide)
+    )
+    (pin "2")
+    (pin "1")
+    (instances
+      (project "diagram_chart"
+        (path "/6dfb841c-0ebb-4587-a5cf-7b85233b045b"
+          (reference "R33") (unit 1)
+        )
+      )
+    )
+  )
   (symbol (lib_id "Device:R") (at 373.38 99.06 0) (mirror x) (unit 1)
     (in_bom yes) (on_board yes) (dnp no) (fields_autoplaced)
@@
     )
   )
+  (symbol (lib_id "Connector:Screw_Terminal_01x02") (at 246.38 266.7 270) (unit 1)
+    (in_bom yes) (on_board yes) (dnp no) (fields_autoplaced)
+    (property "Reference" "NC4" (at 248.92 265.43 90)
+      (effects (font (size 1.27 1.27)) (justify left))
+    )
+    (property "Value" "Screw Terminal" (at 248.92 267.97 90)
+      (effects (font (size 1.27 1.27)) (justify left))
+    )
+    (property "Footprint" "TerminalBlock_Phoenix:TerminalBlock_Phoenix_MPT-0,5-2-2.54_1x02_P2.54mm_Horizontal" (at 246.38 266.7 0)
+      (effects (font (size 1.27 1.27)) hide)
+    )
+    (property "Datasheet" "~" (at 246.38 266.7 0)
+      (effects (font (size 1.27 1.27)) hide)
+    )
+    (pin "1")
+    (pin "2")
+    (instances
+      (project "diagram_chart"
+        (path "/6dfb841c-0ebb-4587-a5cf-7b85233b045b"
+          (reference "NC4") (unit 1)
+        )
+      )
+    )
+  )
   (symbol (lib_id "Switch:SW_SPDT") (at 384.81 176.53 0) (unit 1)
     (in_bom yes) (on_board yes) (dnp no) (fields_autoplaced)
@@
       (effects (font (size 1.27 1.27)) (justify left))
     )
-    (property "Footprint" "Fuse:Fuseholder_Clip-5x20mm_Keystone_3512_Inline_P23.62x7.27mm_D1.02x1.57mm_Horizontal" (at 212.852 45.72 90)
+    (property "Footprint" "Fuse:Fuseholder_Clip-5x20mm_Eaton_1A5601-01_Inline_P20.80x6.76mm_D1.70mm_Horizontal" (at 212.852 45.72 90)
       (effects (font (size 1.27 1.27)) hide)
     )
@@
     )
   )
+  (symbol (lib_id "Connector:Screw_Terminal_01x02") (at 243.84 247.65 90) (unit 1)
+    (in_bom yes) (on_board yes) (dnp no) (fields_autoplaced)
+    (property "Reference" "NC3" (at 248.92 246.38 90)
+      (effects (font (size 1.27 1.27)) (justify right))
+    )
+    (property "Value" "Screw Terminal" (at 248.92 248.92 90)
+      (effects (font (size 1.27 1.27)) (justify right))
+    )
+    (property "Footprint" "TerminalBlock_Phoenix:TerminalBlock_Phoenix_MPT-0,5-2-2.54_1x02_P2.54mm_Horizontal" (at 243.84 247.65 0)
+      (effects (font (size 1.27 1.27)) hide)
+    )
+    (property "Datasheet" "~" (at 243.84 247.65 0)
+      (effects (font (size 1.27 1.27)) hide)
+    )
+    (pin "1")
+    (pin "2")
+    (instances
+      (project "diagram_chart"
+        (path "/6dfb841c-0ebb-4587-a5cf-7b85233b045b"
+          (reference "NC3") (unit 1)
+        )
+      )
+    )
+  )
   (symbol (lib_id "Switch:SW_SPDT") (at 383.54 130.81 0) (unit 1)
     (in_bom yes) (on_board yes) (dnp no)
@@
     )
   )
+  (symbol (lib_id "Connector:Screw_Terminal_01x02") (at 265.43 247.65 90) (unit 1)
+    (in_bom yes) (on_board yes) (dnp no) (fields_autoplaced)
+    (property "Reference" "NC1" (at 270.51 246.38 90)
+      (effects (font (size 1.27 1.27)) (justify right))
+    )
+    (property "Value" "Screw Terminal" (at 270.51 248.92 90)
+      (effects (font (size 1.27 1.27)) (justify right))
+    )
+    (property "Footprint" "TerminalBlock_Phoenix:TerminalBlock_Phoenix_MPT-0,5-2-2.54_1x02_P2.54mm_Horizontal" (at 265.43 247.65 0)
+      (effects (font (size 1.27 1.27)) hide)
+    )
+    (property "Datasheet" "~" (at 265.43 247.65 0)
+      (effects (font (size 1.27 1.27)) hide)
+    )
+    (pin "1")
+    (pin "2")
+    (instances
+      (project "diagram_chart"
+        (path "/6dfb841c-0ebb-4587-a5cf-7b85233b045b"
+          (reference "NC1") (unit 1)
+        )
+      )
+    )
+  )
   (symbol (lib_id "Switch:SW_SPDT") (at 384.81 198.12 0) (unit 1)
     (in_bom yes) (on_board yes) (dnp no) (fields_autoplaced)
@@
     )
   )
+  (symbol (lib_id "Connector:Screw_Terminal_01x02") (at 227.33 57.15 180) (unit 1)
+    (in_bom yes) (on_board yes) (dnp no) (fields_autoplaced)
+    (property "Reference" "RGB2" (at 227.33 48.26 0)
+      (effects (font (size 1.27 1.27)))
+    )
+    (property "Value" "Screw Terminal" (at 227.33 50.8 0)
+      (effects (font (size 1.27 1.27)))
+    )
+    (property "Footprint" "TerminalBlock_Phoenix:TerminalBlock_Phoenix_MPT-0,5-2-2.54_1x02_P2.54mm_Horizontal" (at 227.33 57.15 0)
+      (effects (font (size 1.27 1.27)) hide)
+    )
+    (property "Datasheet" "~" (at 227.33 57.15 0)
+      (effects (font (size 1.27 1.27)) hide)
+    )
+    (pin "1")
+    (pin "2")
+    (instances
+      (project "diagram_chart"
+        (path "/6dfb841c-0ebb-4587-a5cf-7b85233b045b"
+          (reference "RGB2") (unit 1)
+        )
+      )
+    )
+  )
   (symbol (lib_id "Device:LED") (at 101.6 219.71 270) (unit 1)
     (in_bom yes) (on_board yes) (dnp no) (fields_autoplaced)
@@
         )
       )
+    )
+  )
+  (symbol (lib_id "Connector:Screw_Terminal_01x02") (at 267.97 265.43 270) (unit 1)
+    (in_bom yes) (on_board yes) (dnp no) (fields_autoplaced)
+    (property "Reference" "NC2" (at 270.51 264.16 90)
+      (effects (font (size 1.27 1.27)) (justify left))
+    )
+    (property "Value" "Screw Terminal" (at 270.51 266.7 90)
+      (effects (font (size 1.27 1.27)) (justify left))
+    )
+    (property "Footprint" "TerminalBlock_Phoenix:TerminalBlock_Phoenix_MPT-0,5-2-2.54_1x02_P2.54mm_Horizontal" (at 267.97 265.43 0)
+      (effects (font (size 1.27 1.27)) hide)
+    )
+    (property "Datasheet" "~" (at 267.97 265.43 0)
+      (effects (font (size 1.27 1.27)) hide)
+    )
+    (pin "1")
+    (pin "2")
+    (instances
+      (project "diagram_chart"
+        (path "/6dfb841c-0ebb-4587-a5cf-7b85233b045b"
+          (reference "NC2") (unit 1)
+        )
+      )
